File: design.kicad_pcb (KiCad board)
At the start: 2 copper layers, 25 x 22.9 mm, 14 parts, among them J1 Conn_01x02, J2 Conn_01x02, J3 Conn_01x03, J4 Conn_01x03, U1 TPS61099YFFT

Commit message: DEL Template stuff
Parts:
- removed C1, C2, C3, C4: C_Small, Capacitor_SMD:C_0805_2012Metric
- removed J1, J2: Conn_01x02, Connector_PinHeader_2.54mm:PinHeader_1x02_P2.54mm_Vertical
- removed J3, J4: Conn_01x03, Connector_PinHeader_2.54mm:PinHeader_1x03_P2.54mm_Vertical
- removed JP1, JP2: SolderJumper_2_Open, Jumper:SolderJumper-2_P1.3mm_Open_RoundedPad1.0x1.5mm
- removed L1: L_Small, Inductor_SMD:L_1008_2520Metric
- removed R1, R2: R_Small, Resistor_SMD:R_0805_2012Metric
- removed U1: TPS61099YFFT, Converter_DCDC_custom:BGA6N40P3X2_122X88X62N
Routing:
- net En: track 19.9 -> 0.00 mm, vias 1 -> 0
- net Vin: track 14.5 -> 0.00 mm, vias 2 -> 0
- net FB: track 8.82 -> 0.00 mm
- net GND: track 3.05 -> 0.00 mm, vias 36 -> 0
- net Vout: track 2.80 -> 0.00 mm
- net SW: track 2.80 -> 0.00 mm
- removed copper zone on B.Cu, net GND
- removed copper zone on F.Cu, net GND
- removed copper zone on F.Cu, net SW
- removed copper zone on F.Cu, net Vin
- removed copper zone on F.Cu, net Vout
Other:
- board size 25 x 22.9 mm -> 37.7 x 35.3 mm
- board text removed: "EN"
- board text removed: "GND"
- board text removed: "Vin"
- board text removed: "Vout"

Commit message: Update design.kicad_pcb
Parts:
- added C1: C_Small, Capacitor_SMD:C_0805_2012Metric, F.Cu at (121.3, 112.7)
- added C2: C_Small, Capacitor_SMD:C_0805_2012Metric, F.Cu at (125.2, 119.6)
- added C3: C_Small, Capacitor_SMD:C_0805_2012Metric, F.Cu at (128.3, 115.6)
- added C4: C_Small, Capacitor_SMD:C_0805_2012Metric, F.Cu at (130.3, 115.6)
- added C5: C_Small, Capacitor_SMD:C_0805_2012Metric, F.Cu at (132.3, 115.6)
- added L1: WE-MAPI_4020, Snapeda:WE-MAPI_4020_WE-MAPI_4020, F.Cu at (119.7, 117.6)
- added Rosel1: R_Small, Resistor_SMD:R_0805_2012Metric, F.Cu at (125.3, 110.6)
- added U1: TPS61094DSSR, Snapeda:TPS61094DSSR_SON50P300X200X80-13N, F.Cu at (125.0, 115.0)
Other:
- board size 37.7 x 35.3 mm -> 50 x 30 mm

Commit message: update
Parts:
- added NT1: NetTie_2, NetTie:NetTie-2_SMD_Pad0.5mm, F.Cu at (125.5, 115.8)
- moved Rosel1 0.28 mm to (125.0, 110.5)
- moved C2 0.23 mm to (125.0, 119.5)
Connections:
- net Net-(L1-Pad2) renamed /SW
- C1 pad 2: AGND -> GND
- C2 pad 2: AGND -> GND
- C3 pad 2: AGND -> GND
- C4 pad 2: AGND -> GND
- C5 pad 2: AGND -> GND
- U1 pad 13: AGND -> GND
- U1 pad 7: AGND -> GND
Routing:
- net AGND: track 0.00 -> 8.51 mm, vias 0 -> 2
- net Net-(Rosel1-Pad1): track 0.00 -> 3.29 mm
- net Vin: track 0.00 -> 3.27 mm
- added copper zone on F.Cu, net /SW
- added copper zone on B.Cu, net GND
- added copper zone on F.Cu, net GND
- added copper zone on F.Cu, net Vin
- added copper zone on F.Cu, net Vout
