File: design.kicad_pcb (KiCad board)
At the start: 2 copper layers, 50 x 30 mm, 9 parts, among them U1 TPS61094DSSR

Commit message: update
Parts:
- NT1: moved to B.Cu
- moved NT1 2.02 mm to (127.0, 114.3), turned to 90 degrees
Connections:
- C1 pad 1: Vin -> EN
- C2 pad 1: Vin -> EN
- L1 pad 1: Vin -> EN
- U1 pad 2: Mode -> EN
- U1 pad 4: Vin -> EN
- U1 pad 6: Vin -> EN
- U1 pad 8: AGND -> GND
Routing:
- net EN: track 0.00 -> 15.1 mm
- net Vin: track 3.27 -> 0.00 mm
- net AGND: track 8.51 -> 5.52 mm, vias 2 -> 1
- net GND: track 0.00 -> 1.84 mm, vias 0 -> 21
- added copper zone on F.Cu, net EN
- removed copper zone on F.Cu, net Vin

Commit message: update
Parts:
- added J1: Conn_02x02_Counter_Clockwise, Connector_PinHeader_2.54mm:PinHeader_2x02_P2.54mm_Vertical, F.Cu at (112.3, 121.8)
- added J2: Conn_02x02_Counter_Clockwise, Connector_PinHeader_2.54mm:PinHeader_2x02_P2.54mm_Vertical, F.Cu at (141.2, 116.8)
- added TP1: Vin, TestPoint:TestPoint_Pad_D3.0mm, F.Cu at (105.5, 116.6)
- added TP2: Vout, TestPoint:TestPoint_Pad_D3.0mm, F.Cu at (145.8, 112.7)
- added TP3: GND, TestPoint:TestPoint_Pad_D3.0mm, F.Cu at (105.8, 126.6)
- added TP4: GND, TestPoint:TestPoint_Pad_D3.0mm, F.Cu at (145.8, 126.5)
- added TP5: RCWCTE, Snapeda:RCWCTE_TP420X150, F.Cu at (140.0, 110.2)
- added TP6: RCWCTE, Snapeda:RCWCTE_TP420X150, F.Cu at (140.0, 120.8)
- added TP7: RCWCTE, Snapeda:RCWCTE_TP420X150, F.Cu at (111.3, 113.2)
- added TP8: RCWCTE, Snapeda:RCWCTE_TP420X150, F.Cu at (111.3, 104.3)

Commit message: Update design.kicad_pcb
Parts:
- moved TP3 2.78 mm to (103.0, 127.0)
- moved TP4 1.27 mm to (147.0, 127.0)
Routing:
- net GND: vias 21 -> 33
Changed lines of the file:
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@@
     (property "Sheetname" "")
     (attr smd)
-    (fp_text reference "TP8" (at 3 0 90) (layer "F.SilkS")
+    (fp_text reference "TP8" (at -2.85 0 90) (layer "F.SilkS")
       (effects (font (size 0.64 0.64) (thickness 0.15)))
     )
@@
       (effects (font (size 0.64 0.64) (thickness 0.15)))
     )
-    (fp_text user "GND" (at 0 0 unlocked) (layer "F.SilkS")
+    (fp_text user "GND" (at 0 2.05 unlocked) (layer "F.SilkS")
       (effects (font (size 1 1) (thickness 0.15)))
     )
@@
   )
   (footprint "TestPoint:TestPoint_Pad_D3.0mm" (layer "F.Cu")
-    (at 105.75 126.6 180)
+    (at 103 127 180)
     (descr "SMD pad as test Point, diameter 3.0mm")
     (tags "test point SMD pad")
@@
       (effects (font (size 0.64 0.64) (thickness 0.15)))
     )
-    (fp_text user "Vout" (at 0 0 unlocked) (layer "F.SilkS")
+    (fp_text user "Vout" (at 0 1.7 unlocked) (layer "F.SilkS")
       (effects (font (size 1 1) (thickness 0.15)))
     )
@@
   )
   (footprint "TestPoint:TestPoint_Pad_D3.0mm" (layer "F.Cu")
-    (at 145.85 126.45 180)
+    (at 147 127 180)
     (descr "SMD pad as test Point, diameter 3.0mm")
     (tags "test point SMD pad")
@@
       (effects (font (size 0.64 0.64) (thickness 0.15)))
     )
-    (fp_text user "Vin" (at 0 0 unlocked) (layer "F.SilkS")
+    (fp_text user "Vin" (at 0 1.8 unlocked) (layer "F.SilkS")
       (effects (font (size 1 1) (thickness 0.15)))
     )
@@
       (effects (font (size 0.64 0.64) (thickness 0.15)))
     )
-    (fp_text user "GND" (at 0 0 unlocked) (layer "F.SilkS")
+    (fp_text user "GND" (at 0 1.95 unlocked) (layer "F.SilkS")
       (effects (font (size 1 1) (thickness 0.15)))
     )
@@
   )
   (gr_rect (start 100 100) (end 150 130) (layer "Edge.Cuts") (width 0.05) (fill none))
-  (gr_text "<<project_name>>\n<<ID>>\n<<version>>\n<<date>>\n<<hash>>\n<<website_link>>" (at 225.75 151) (layer "F.SilkS")
-    (effects (font (size 1 1) (thickness 0.15)))
+  (gr_text "<<project_name>>\n<<ID>>\n<<version>>\n<<date>>\n<<hash>>\n<<website_link>>" (at 136 106) (layer "B.SilkS")
+    (effects (font (size 1 1) (thickness 0.15)) (justify mirror))
   )
   (segment (start 126.01 110.5975) (end 125.9125 110.5) (width 0.25) (layer "F.Cu") (net 1))
@@
   (segment (start 115.15 121) (end 115.15 119.95) (width 0.25) (layer "F.Cu") (net 4))
   (segment (start 126.95 115.75) (end 126.01 115.75) (width 0.25) (layer "F.Cu") (net 6))
+  (via (at 115 104) (size 0.8) (drill 0.4) (layers "F.Cu" "B.Cu") (free) (net 6))
+  (via (at 107 127) (size 0.8) (drill 0.4) (layers "F.Cu" "B.Cu") (free) (net 6))
   (via (at 122.2 109.2) (size 0.8) (drill 0.4) (layers "F.Cu" "B.Cu") (free) (net 6))
+  (via (at 144 127) (size 0.8) (drill 0.4) (layers "F.Cu" "B.Cu") (free) (net 6))
   (via (at 129.2 119) (size 0.8) (drill 0.4) (layers "F.Cu" "B.Cu") (free) (net 6))
   (via (at 131.2 118) (size 0.8) (drill 0.4) (layers "F.Cu" "B.Cu") (free) (net 6))
@@
   (via (at 126.95 115.75) (size 0.8) (drill 0.4) (layers "F.Cu" "B.Cu") (net 6))
   (via (at 132.2 118) (size 0.8) (drill 0.4) (layers "F.Cu" "B.Cu") (free) (net 6))
+  (via (at 106 128) (size 0.8) (drill 0.4) (layers "F.Cu" "B.Cu") (free) (net 6))
+  (via (at 116 104) (size 0.8) (drill 0.4) (layers "F.Cu" "B.Cu") (free) (net 6))
+  (via (at 106 127) (size 0.8) (drill 0.4) (layers "F.Cu" "B.Cu") (free) (net 6))
   (via (at 128.2 118) (size 0.8) (drill 0.4) (layers "F.Cu" "B.Cu") (free) (net 6))
   (via (at 127.2 119) (size 0.8) (drill 0.4) (layers "F.Cu" "B.Cu") (free) (net 6))
@@
   (via (at 130.2 119) (size 0.8) (drill 0.4) (layers "F.Cu" "B.Cu") (free) (net 6))
   (via (at 127.2 118) (size 0.8) (drill 0.4) (layers "F.Cu" "B.Cu") (free) (net 6))
+  (via (at 143 128) (size 0.8) (drill 0.4) (layers "F.Cu" "B.Cu") (free) (net 6))
+  (via (at 107 128) (size 0.8) (drill 0.4) (layers "F.Cu" "B.Cu") (free) (net 6))
+  (via (at 116 105) (size 0.8) (drill 0.4) (layers "F.Cu" "B.Cu") (free) (net 6))
+  (via (at 144 128) (size 0.8) (drill 0.4) (layers "F.Cu" "B.Cu") (free) (net 6))
+  (via (at 143 127) (size 0.8) (drill 0.4) (layers "F.Cu" "B.Cu") (free) (net 6))
   (via (at 133.2 118) (size 0.8) (drill 0.4) (layers "F.Cu" "B.Cu") (free) (net 6))
+  (via (at 115 105) (size 0.8) (drill 0.4) (layers "F.Cu" "B.Cu") (free) (net 6))
   (via (at 129.2 118) (size 0.8) (drill 0.4) (layers "F.Cu" "B.Cu") (free) (net 6))
   (via (at 121.2 109.2) (size 0.8) (drill 0.4) (layers "F.Cu" "B.Cu") (free) (net 6))

Commit message: update
Parts:
- C1: value C_Small -> 2.2uF
- C3: value C_Small -> 22uF
- C4, C5: value C_Small -> DNP
- L1: value WE-MAPI_4020 -> 74438356022
Connections:
- net EN renamed Vin
Other:
- outline, holes or cut-outs redrawn
- board text added: "Boost Converter with Bypass Mod"
- board text added: "Rosel 4.75k - 3.3V 205k - 5V"
Changed lines of the file:
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@@
   (net 2 "Vout")
   (net 3 "Net-(Rosel1-Pad1)")
-  (net 4 "EN")
+  (net 4 "Vin")
   (net 5 "/SW")
   (net 6 "GND")
@@
       (net 3 "Net-(Rosel1-Pad1)") (pinfunction "OSEL") (pintype "input") (solder_mask_margin 0.102))
     (pad "2" smd roundrect (at -1.01 -0.75) (size 0.71 0.27) (layers "F.Cu" "F.Paste" "F.Mask") (roundrect_rratio 0.125)
-      (net 4 "EN") (pinfunction "MODE") (pintype "input") (solder_mask_margin 0.102))
+      (net 4 "Vin") (pinfunction "MODE") (pintype "input") (solder_mask_margin 0.102))
     (pad "3" smd roundrect (at -1.01 -0.25) (size 0.71 0.27) (layers "F.Cu" "F.Paste" "F.Mask") (roundrect_rratio 0.125)
-      (net 4 "EN") (pinfunction "EN") (pintype "input") (solder_mask_margin 0.102))
+      (net 4 "Vin") (pinfunction "EN") (pintype "input") (solder_mask_margin 0.102))
     (pad "4" smd roundrect (at -1.01 0.25) (size 0.71 0.27) (layers "F.Cu" "F.Paste" "F.Mask") (roundrect_rratio 0.125)
-      (net 4 "EN") (pinfunction "VIN") (pintype "input") (solder_mask_margin 0.102))
+      (net 4 "Vin") (pinfunction "VIN") (pintype "input") (solder_mask_margin 0.102))
     (pad "5" smd roundrect (at -1.01 0.75) (size 0.71 0.27) (layers "F.Cu" "F.Paste" "F.Mask") (roundrect_rratio 0.125)
       (net 5 "/SW") (pinfunction "SW") (pintype "passive") (solder_mask_margin 0.102))
     (pad "6" smd roundrect (at -1.01 1.25) (size 0.71 0.27) (layers "F.Cu" "F.Paste" "F.Mask") (roundrect_rratio 0.125)
-      (net 4 "EN") (pinfunction "SUP") (pintype "input") (solder_mask_margin 0.102))
+      (net 4 "Vin") (pinfunction "SUP") (pintype "input") (solder_mask_margin 0.102))
     (pad "7" smd roundrect (at 1.01 1.25) (size 0.71 0.27) (layers "F.Cu" "F.Paste" "F.Mask") (roundrect_rratio 0.125)
       (net 6 "GND") (pinfunction "PGND") (pintype "power_in") (solder_mask_margin 0.102))
@@
     (fp_line (start 1 0.625) (end -1 0.625) (layer "F.Fab") (width 0.1))
     (pad "1" smd roundrect (at -0.95 0) (size 1 1.45) (layers "F.Cu" "F.Paste" "F.Mask") (roundrect_rratio 0.25)
-      (net 4 "EN") (pintype "passive"))
+      (net 4 "Vin") (pintype "passive"))
     (pad "2" smd roundrect (at 0.95 0) (size 1 1.45) (layers "F.Cu" "F.Paste" "F.Mask") (roundrect_rratio 0.25)
       (net 6 "GND") (pintype "passive"))
@@
       (net 6 "GND") (pinfunction "Pin_2") (pintype "passive"))
     (pad "3" thru_hole oval (at 0 2.54 180) (size 1.7 1.7) (drill 1) (layers *.Cu *.Mask)
-      (net 4 "EN") (pinfunction "Pin_3") (pintype "passive"))
+      (net 4 "Vin") (pinfunction "Pin_3") (pintype "passive"))
     (pad "4" thru_hole oval (at 2.54 2.54 180) (size 1.7 1.7) (drill 1) (layers *.Cu *.Mask)
-      (net 4 "EN") (pinfunction "Pin_4") (pintype "passive"))
+      (net 4 "Vin") (pinfunction "Pin_4") (pintype "passive"))
     (model "${KICAD6_3DMODEL_DIR}/Connector_PinHeader_2.54mm.3dshapes/PinHeader_2x02_P2.54mm_Vertical.wrl"
       (offset (xyz 0 0 0))
@@
       (effects (font (size 1 1) (thickness 0.15)))
     )
-    (fp_text value "WE-MAPI_4020" (at 0 3.365) (layer "F.Fab")
+    (fp_text value "74438356022" (at 0 3.365) (layer "F.Fab")
       (effects (font (size 1 1) (thickness 0.15)))
     )
@@
     (fp_line (start -2.05 -2.05) (end 2.05 -2.05) (layer "F.Fab") (width 0.1))
     (pad "1" smd rect (at -1.185 0) (size 0.98 3.7) (layers "F.Cu" "F.Paste" "F.Mask")
-      (net 4 "EN") (pintype "passive") (solder_mask_margin 0.102))
+      (net 4 "Vin") (pintype "passive") (solder_mask_margin 0.102))
     (pad "2" smd rect (at 1.185 0) (size 0.98 3.7) (layers "F.Cu" "F.Paste" "F.Mask")
       (net 5 "/SW") (pintype "passive") (solder_mask_margin 0.102))
@@
     (property "Sheetfile" "design.kicad_sch")
     (property "Sheetname" "")
-    (attr smd)
+    (property "exclude_from_bom" "")
+    (attr smd exclude_from_bom)
     (fp_text reference "C5" (at -2.6 0.01 90) (layer "F.SilkS")
       (effects (font (size 1 1) (thickness 0.15)))
     )
-    (fp_text value "C_Small" (at 0 1.68 90) (layer "F.Fab")
+    (fp_text value "DNP" (at 0 1.68 90) (layer "F.Fab")
       (effects (font (size 1 1) (thickness 0.15)))
     )
@@
     (fp_circle (center 0 0) (end 2 0) (layer "F.CrtYd") (width 0.05) (fill none))
     (pad "1" smd circle (at 0 0) (size 3 3) (layers "F.Cu" "F.Mask")
-      (net 4 "EN") (pinfunction "1") (pintype "passive"))
+      (net 4 "Vin") (pinfunction "1") (pintype "passive"))
   )
   (footprint "Snapeda:RCWCTE_TP420X150" (layer "F.Cu")
@@
     (fp_line (start 1.6 -0.8) (end 1.6 0.8) (layer "F.Fab") (width 0.127))
     (pad "1" smd rect (at 0 0) (size 4.2 1.5) (layers "F.Cu" "F.Paste" "F.Mask")
-      (net 4 "EN") (pintype "passive") (solder_mask_margin 0.102))
+      (net 4 "Vin") (pintype "passive") (solder_mask_margin 0.102))
     (model "${KICAD_3RD_PARTY}/Snapeda.3dshapes/RCWCTE.step"
       (offset (xyz 0 0 0))
@@
       (effects (font (size 1 1) (thickness 0.15)))
     )
-    (fp_text value "C_Small" (at 0 1.68 90) (layer "F.Fab")
+    (fp_text value "22uF" (at 0 1.68 90) (layer "F.Fab")
       (effects (font (size 1 1) (thickness 0.15)))
     )
@@
       (effects (font (size 1 1) (thickness 0.15)))
     )
-    (fp_text value "C_Small" (at 0 1.68 90) (layer "F.Fab")
+    (fp_text value "2.2uF" (at 0 1.68 90) (layer "F.Fab")
       (effects (font (size 1 1) (thickness 0.15)))
     )
@@
     (fp_line (start 1 0.625) (end -1 0.625) (layer "F.Fab") (width 0.1))
     (pad "1" smd roundrect (at -0.95 0 90) (size 1 1.45) (layers "F.Cu" "F.Paste" "F.Mask") (roundrect_rratio 0.25)
-      (net 4 "EN") (pintype "passive"))
+      (net 4 "Vin") (pintype "passive"))
     (pad "2" smd roundrect (at 0.95 0 90) (size 1 1.45) (layers "F.Cu" "F.Paste" "F.Mask") (roundrect_rratio 0.25)
       (net 6 "GND") (pintype "passive"))
@@
     (property "Sheetfile" "design.kicad_sch")
     (property "Sheetname" "")
-    (attr smd)
+    (property "exclude_from_bom" "")
+    (attr smd exclude_from_bom)
     (fp_text reference "C4" (at -2.6 0.01 90) (layer "F.SilkS")
       (effects (font (size 1 1) (thickness 0.15)))
     )
-    (fp_text value "C_Small" (at 0 1.68 90) (layer "F.Fab")
+    (fp_text value "DNP" (at 0 1.68 90) (layer "F.Fab")
       (effects (font (size 1 1) (thickness 0.15)))
     )
@@
       (net 1 "AGND") (pinfunction "2") (pintype "passive"))
   )
-  (gr_rect (start 100 100) (end 150 130) (layer "Edge.Cuts") (width 0.05) (fill none))
+  (gr_arc (start 103 130) (mid 100.87868 129.12132) (end 100 127) (layer "Edge.Cuts") (width 0.05))
+  (gr_arc (start 100 103) (mid 100.87868 100.87868) (end 103 100) (layer "Edge.Cuts") (width 0.05))
+  (gr_line (start 100 103) (end 100 127) (layer "Edge.Cuts") (width 0.05))
+  (gr_line (start 150 127) (end 150 103) (layer "Edge.Cuts") (width 0.05))
+  (gr_arc (start 147 100) (mid 149.12132 100.87868) (end 150 103) (layer "Edge.Cuts") (width 0.05))
+  (gr_line (start 103 130) (end 147 130) (layer "Edge.Cuts") (width 0.05))
+  (gr_line (start 147 100) (end 103 100) (layer "Edge.Cuts") (width 0.05))
+  (gr_arc (start 150 127) (mid 149.12132 129.12132) (end 147 130) (layer "Edge.Cuts") (width 0.05))
   (gr_text "<<project_name>>\n<<ID>>\n<<version>>\n<<date>>\n<<hash>>\n<<website_link>>" (at 136 106) (layer "B.SilkS")
     (effects (font (size 1 1) (thickness 0.15)) (justify mirror))
+  )
+  (gr_text "Rosel\n4.75k - 3.3V\n205k - 5V " (at 124.5 104) (layer "F.SilkS")
+    (effects (font (size 1 1) (thickness 0.15)))
+  )
+  (gr_text "Boost Converter with Bypass Mod" (at 125 127) (layer "F.SilkS")
+    (effects (font (size 1 1) (thickness 0.15)))
   )
   (segment (start 126.01 110.5975) (end 125.9125 110.5) (width 0.25) (layer "F.Cu") (net 1))
@@
     )
   )
-  (zone (net 4) (net_name "EN") (layer "F.Cu") (hatch edge 0.508)
+  (zone (net 4) (net_name "Vin") (layer "F.Cu") (hatch edge 0.508)
     (priority 1)
     (connect_pads yes (clearance 0.2))
