File: design.kicad_sch (KiCad schematic)
At the start: 0 parts

Commit message: Update design.kicad_sch
Parts:
- added C1, C2, C3, C4, C5: C_Small, Capacitor_SMD:C_0805_2012Metric, symbol Device:C_Small
- added L1: WE-MAPI_4020, Snapeda:WE-MAPI_4020_WE-MAPI_4020, symbol Snapeda:WE-MAPI_4020
- added Rosel1: R_Small, Resistor_SMD:R_0805_2012Metric, symbol Device:R_Small
- added U1: TPS61094DSSR, Snapeda:TPS61094DSSR_SON50P300X200X80-13N, symbol Snapeda:TPS61094DSSR
Connections:
- new net: L1.2, U1.5 (SW)
- new net: Rosel1.1, U1.1 (OSEL)
- new net EN: U1.3 (EN)
- new net GND: C1.2, C2.2, C3.2, C4.2, C5.2, Rosel1.2, U1.11 (ICHG), U1.12 (VCHG), U1.13 (EXP), U1.7 (PGND), U1.8 (AGND)
- new net Mode: U1.2 (MODE)
- new net Vin: C1.1, C2.1, L1.1, U1.4 (VIN), U1.6 (SUP)
- new net Vout: C3.1, C4.1, C5.1, U1.10 (VOUT), U1.9 (VOUT)

Commit message: update
Parts:
- added NT1: NetTie_2, NetTie:NetTie-2_SMD_Pad0.5mm, symbol Device:NetTie_2
Connections:
- net GND: now also NT1.1; no longer Rosel1.2, U1.11 (ICHG), U1.12 (VCHG), U1.8 (AGND)
- net SW: now reaches L1.2, U1.5 (SW)
- new net AGND: NT1.2, Rosel1.2, U1.11 (ICHG), U1.12 (VCHG), U1.8 (AGND)
Changed lines of the file:
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@@
   (junction (at 180.34 71.12) (diameter 0) (color 0 0 0 0)
   )
-  (junction (at 165.1 96.52) (diameter 0) (color 0 0 0 0)
-  )
-  (junction (at 167.64 99.06) (diameter 0) (color 0 0 0 0)
-  )
   (junction (at 165.1 88.9) (diameter 0) (color 0 0 0 0)
   )
@@
   (junction (at 91.44 71.12) (diameter 0) (color 0 0 0 0)
   )
+  (junction (at 165.1 99.06) (diameter 0) (color 0 0 0 0)
+  )
   (junction (at 187.96 78.74) (diameter 0) (color 0 0 0 0)
   )
@@
     (stroke (width 0) (type default) (color 0 0 0 0))
   )
-  (wire (pts (xy 162.56 99.06) (xy 167.64 99.06))
+  (wire (pts (xy 162.56 99.06) (xy 165.1 99.06))
+    (stroke (width 0) (type default) (color 0 0 0 0))
+  )
+  (wire (pts (xy 172.72 99.06) (xy 165.1 99.06))
     (stroke (width 0) (type default) (color 0 0 0 0))
   )
@@
     (stroke (width 0) (type default) (color 0 0 0 0))
   )
-  (wire (pts (xy 167.64 99.06) (xy 167.64 104.14))
+  (wire (pts (xy 162.56 93.98) (xy 172.72 93.98))
+    (stroke (width 0) (type default) (color 0 0 0 0))
+  )
+  (wire (pts (xy 165.1 99.06) (xy 165.1 104.14))
     (stroke (width 0) (type default) (color 0 0 0 0))
   )
@@
     (stroke (width 0) (type default) (color 0 0 0 0))
   )
-  (wire (pts (xy 165.1 96.52) (xy 167.64 96.52))
+  (wire (pts (xy 172.72 93.98) (xy 172.72 99.06))
     (stroke (width 0) (type default) (color 0 0 0 0))
   )
@@
     (stroke (width 0) (type default) (color 0 0 0 0))
   )
-  (wire (pts (xy 167.64 96.52) (xy 167.64 99.06))
-    (stroke (width 0) (type default) (color 0 0 0 0))
-  )
   (wire (pts (xy 91.44 96.52) (xy 96.52 96.52))
     (stroke (width 0) (type default) (color 0 0 0 0))
@@
     (stroke (width 0) (type default) (color 0 0 0 0))
   )
-  (wire (pts (xy 165.1 93.98) (xy 165.1 96.52))
-    (stroke (width 0) (type default) (color 0 0 0 0))
-  )
   (wire (pts (xy 167.64 78.74) (xy 167.64 81.28))
     (stroke (width 0) (type default) (color 0 0 0 0))
@@
     (stroke (width 0) (type default) (color 0 0 0 0))
   )
-  (wire (pts (xy 162.56 93.98) (xy 165.1 93.98))
+  (wire (pts (xy 178.435 95.885) (xy 182.245 95.885))
     (stroke (width 0) (type default) (color 0 0 0 0))
   )
@@
     (stroke (width 0) (type default) (color 0 0 0 0))
   )
-  (wire (pts (xy 162.56 96.52) (xy 165.1 96.52))
-    (stroke (width 0) (type default) (color 0 0 0 0))
-  )
   (wire (pts (xy 180.34 76.2) (xy 180.34 78.74))
     (stroke (width 0) (type default) (color 0 0 0 0))
@@
   (wire (pts (xy 187.96 78.74) (xy 195.58 78.74))
     (stroke (width 0) (type default) (color 0 0 0 0))
+  )
+  (label "SUP" (at 120.015 81.28 0)
+    (effects (font (size 1.27 1.27)) (justify left bottom))
+  )
+  (label "SW" (at 120.015 76.2 0)
+    (effects (font (size 1.27 1.27)) (justify left bottom))
   )
   (global_label "EN" (shape input) (at 127 88.9 180) (fields_autoplaced)
@@
     )
   )
-  (global_label "AGND" (shape input) (at 167.64 96.52 0) (fields_autoplaced)
+  (global_label "AGND" (shape input) (at 162.56 96.52 0) (fields_autoplaced)
     (effects (font (size 1.27 1.27)) (justify left))
-    (property "Referenzen zwischen Schaltplänen" "${INTERSHEET_REFS}" (id 0) (at 174.9232 96.4406 0)
+    (property "Referenzen zwischen Schaltplänen" "${INTERSHEET_REFS}" (id 0) (at 169.8432 96.4406 0)
+      (effects (font (size 1.27 1.27)) (justify left) hide)
+    )
+  )
+  (global_label "AGND" (shape input) (at 187.325 95.885 0) (fields_autoplaced)
+    (effects (font (size 1.27 1.27)) (justify left))
+    (property "Referenzen zwischen Schaltplänen" "${INTERSHEET_REFS}" (id 0) (at 194.6082 95.8056 0)
       (effects (font (size 1.27 1.27)) (justify left) hide)
     )
@@
     (pin "2")
   )
+  (symbol (lib_id "power:GND") (at 178.435 95.885 0) (unit 1)
+    (in_bom yes) (on_board yes) (fields_autoplaced)
+    (property "Reference" "#PWR?" (id 0) (at 178.435 102.235 0)
+      (effects (font (size 1.27 1.27)) hide)
+    )
+    (property "Value" "GND" (id 1) (at 178.435 100.965 0))
+    (property "Footprint" "" (id 2) (at 178.435 95.885 0)
+      (effects (font (size 1.27 1.27)) hide)
+    )
+    (property "Datasheet" "" (id 3) (at 178.435 95.885 0)
+      (effects (font (size 1.27 1.27)) hide)
+    )
+    (pin "1")
+  )
   (symbol (lib_id "power:GND") (at 195.58 81.28 0) (unit 1)
     (in_bom yes) (on_board yes) (fields_autoplaced)
@@
     (pin "1")
   )
-  (symbol (lib_id "power:GND") (at 167.64 104.14 0) (unit 1)
-    (in_bom yes) (on_board yes) (fields_autoplaced)
-    (property "Reference" "#PWR0104" (id 0) (at 167.64 110.49 0)
-      (effects (font (size 1.27 1.27)) hide)
-    )
-    (property "Value" "GND" (id 1) (at 167.64 109.22 0))
-    (property "Footprint" "" (id 2) (at 167.64 104.14 0)
-      (effects (font (size 1.27 1.27)) hide)
-    )
-    (property "Datasheet" "" (id 3) (at 167.64 104.14 0)
+  (symbol (lib_id "Device:NetTie_2") (at 184.785 95.885 0) (unit 1)
+    (in_bom no) (on_board yes) (fields_autoplaced)
+    (property "Reference" "NT1" (id 0) (at 184.785 90.805 0))
+    (property "Value" "NetTie_2" (id 1) (at 184.785 93.345 0))
+    (property "Footprint" "NetTie:NetTie-2_SMD_Pad0.5mm" (id 2) (at 184.785 95.885 0)
+      (effects (font (size 1.27 1.27)) hide)
+    )
+    (property "Datasheet" "~" (id 3) (at 184.785 95.885 0)
+      (effects (font (size 1.27 1.27)) hide)
+    )
+    (pin "1")
+    (pin "2")
+  )
+  (symbol (lib_id "power:GND") (at 165.1 104.14 0) (unit 1)
+    (in_bom yes) (on_board yes) (fields_autoplaced)
+    (property "Reference" "#PWR0104" (id 0) (at 165.1 110.49 0)
+      (effects (font (size 1.27 1.27)) hide)
+    )
+    (property "Value" "GND" (id 1) (at 165.1 109.22 0))
+    (property "Footprint" "" (id 2) (at 165.1 104.14 0)
+      (effects (font (size 1.27 1.27)) hide)
+    )
+    (property "Datasheet" "" (id 3) (at 165.1 104.14 0)
       (effects (font (size 1.27 1.27)) hide)
     )
@@
       (reference "#PWR0104") (unit 1) (value "GND") (footprint "")
     )
+    (path "/95e1eb76-8da9-4d97-8379-8facac6c427d"
+      (reference "#PWR?") (unit 1) (value "GND") (footprint "")
+    )
     (path "/ca007935-a432-42f1-b756-6e4a1ace9956"
       (reference "C1") (unit 1) (value "C_Small") (footprint "Capacitor_SMD:C_0805_2012Metric")
@@
       (reference "L1") (unit 1) (value "WE-MAPI_4020") (footprint "Snapeda:WE-MAPI_4020_WE-MAPI_4020")
     )
+    (path "/b0f91be2-7d60-44ef-8328-61d7e6e65bb6"
+      (reference "NT1") (unit 1) (value "NetTie_2") (footprint "NetTie:NetTie-2_SMD_Pad0.5mm")
+    )
     (path "/8d96c754-c2de-4e99-9f69-81192f00f7ae"

Commit message: Update design.kicad_sch
Connections:
- net Mode is gone; now on net EN: U1.2 (MODE)
- net Vin is gone; now on net EN: C1.1, C2.1, L1.1, U1.4 (VIN), U1.6 (SUP)
Changed lines of the file:
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@@
   (junction (at 195.58 78.74) (diameter 0) (color 0 0 0 0)
   )
+  (junction (at 165.1 102.87) (diameter 0) (color 0 0 0 0)
+  )
   (junction (at 180.34 71.12) (diameter 0) (color 0 0 0 0)
   )
+  (junction (at 147.32 127) (diameter 0) (color 0 0 0 0)
+  )
   (junction (at 165.1 88.9) (diameter 0) (color 0 0 0 0)
   )
   (junction (at 91.44 96.52) (diameter 0) (color 0 0 0 0)
   )
+  (junction (at 97.155 71.12) (diameter 0) (color 0 0 0 0)
+  )
   (junction (at 195.58 71.12) (diameter 0) (color 0 0 0 0)
   )
@@
     (stroke (width 0) (type default) (color 0 0 0 0))
   )
+  (wire (pts (xy 97.155 71.12) (xy 104.14 71.12))
+    (stroke (width 0) (type default) (color 0 0 0 0))
+  )
   (wire (pts (xy 167.64 86.36) (xy 167.64 88.9))
     (stroke (width 0) (type default) (color 0 0 0 0))
@@
     (stroke (width 0) (type default) (color 0 0 0 0))
   )
+  (wire (pts (xy 147.32 127) (xy 147.32 129.54))
+    (stroke (width 0) (type default) (color 0 0 0 0))
+  )
   (wire (pts (xy 172.72 99.06) (xy 165.1 99.06))
     (stroke (width 0) (type default) (color 0 0 0 0))
   )
-  (wire (pts (xy 91.44 71.12) (xy 104.14 71.12))
+  (wire (pts (xy 91.44 71.12) (xy 97.155 71.12))
     (stroke (width 0) (type default) (color 0 0 0 0))
   )
@@
     (stroke (width 0) (type default) (color 0 0 0 0))
   )
+  (wire (pts (xy 147.32 127) (xy 153.035 127))
+    (stroke (width 0) (type default) (color 0 0 0 0))
+  )
   (wire (pts (xy 119.38 104.14) (xy 91.44 104.14))
     (stroke (width 0) (type default) (color 0 0 0 0))
@@
     (stroke (width 0) (type default) (color 0 0 0 0))
   )
-  (wire (pts (xy 165.1 99.06) (xy 165.1 104.14))
+  (wire (pts (xy 165.1 99.06) (xy 165.1 102.87))
     (stroke (width 0) (type default) (color 0 0 0 0))
   )
@@
     (stroke (width 0) (type default) (color 0 0 0 0))
   )
+  (wire (pts (xy 140.97 127) (xy 147.32 127))
+    (stroke (width 0) (type default) (color 0 0 0 0))
+  )
   (wire (pts (xy 119.38 111.76) (xy 119.38 114.3))
     (stroke (width 0) (type default) (color 0 0 0 0))
@@
     (stroke (width 0) (type default) (color 0 0 0 0))
   )
+  (wire (pts (xy 165.1 102.87) (xy 165.1 104.14))
+    (stroke (width 0) (type default) (color 0 0 0 0))
+  )
   (wire (pts (xy 91.44 96.52) (xy 96.52 96.52))
     (stroke (width 0) (type default) (color 0 0 0 0))
@@
   )
   (wire (pts (xy 167.64 78.74) (xy 167.64 81.28))
+    (stroke (width 0) (type default) (color 0 0 0 0))
+  )
+  (wire (pts (xy 147.32 129.54) (xy 140.97 129.54))
     (stroke (width 0) (type default) (color 0 0 0 0))
   )
@@
     )
   )
+  (global_label "EN" (shape input) (at 140.97 129.54 180) (fields_autoplaced)
+    (effects (font (size 1.27 1.27)) (justify right))
+    (property "Referenzen zwischen Schaltplänen" "${INTERSHEET_REFS}" (id 0) (at 136.1663 129.4606 0)
+      (effects (font (size 1.27 1.27)) (justify right) hide)
+    )
+  )
   (global_label "Mode" (shape input) (at 127 86.36 180) (fields_autoplaced)
     (effects (font (size 1.27 1.27)) (justify right))
@@
     )
   )
+  (global_label "Vin" (shape input) (at 153.035 127 0) (fields_autoplaced)
+    (effects (font (size 1.27 1.27)) (justify left))
+    (property "Referenzen zwischen Schaltplänen" "${INTERSHEET_REFS}" (id 0) (at 158.2016 127.0794 0)
+      (effects (font (size 1.27 1.27)) (justify left) hide)
+    )
+  )
   (global_label "AGND" (shape input) (at 162.56 96.52 0) (fields_autoplaced)
     (effects (font (size 1.27 1.27)) (justify left))
@@
     )
   )
+  (global_label "Mode" (shape input) (at 140.97 127 180) (fields_autoplaced)
+    (effects (font (size 1.27 1.27)) (justify right))
+    (property "Referenzen zwischen Schaltplänen" "${INTERSHEET_REFS}" (id 0) (at 133.8077 126.9206 0)
+      (effects (font (size 1.27 1.27)) (justify right) hide)
+    )
+  )
+  (symbol (lib_id "power:PWR_FLAG") (at 165.1 102.87 270) (unit 1)
+    (in_bom yes) (on_board yes) (fields_autoplaced)
+    (property "Reference" "#FLG01" (id 0) (at 167.005 102.87 0)
+      (effects (font (size 1.27 1.27)) hide)
+    )
+    (property "Value" "PWR_FLAG" (id 1) (at 168.91 102.8699 90)
+      (effects (font (size 1.27 1.27)) (justify left))
+    )
+    (property "Footprint" "" (id 2) (at 165.1 102.87 0)
+      (effects (font (size 1.27 1.27)) hide)
+    )
+    (property "Datasheet" "~" (id 3) (at 165.1 102.87 0)
+      (effects (font (size 1.27 1.27)) hide)
+    )
+    (pin "1")
+  )
   (symbol (lib_id "Device:C_Small") (at 180.34 73.66 0) (unit 1)
     (in_bom yes) (on_board yes) (fields_autoplaced)
@@
   (symbol (lib_id "power:GND") (at 178.435 95.885 0) (unit 1)
     (in_bom yes) (on_board yes) (fields_autoplaced)
-    (property "Reference" "#PWR?" (id 0) (at 178.435 102.235 0)
+    (property "Reference" "#PWR0105" (id 0) (at 178.435 102.235 0)
       (effects (font (size 1.27 1.27)) hide)
     )
@@
     )
     (property "Datasheet" "" (id 3) (at 178.435 95.885 0)
+      (effects (font (size 1.27 1.27)) hide)
+    )
+    (pin "1")
+  )
+  (symbol (lib_id "power:PWR_FLAG") (at 97.155 71.12 0) (unit 1)
+    (in_bom yes) (on_board yes) (fields_autoplaced)
+    (property "Reference" "#FLG0101" (id 0) (at 97.155 69.215 0)
+      (effects (font (size 1.27 1.27)) hide)
+    )
+    (property "Value" "PWR_FLAG" (id 1) (at 97.155 66.04 0))
+    (property "Footprint" "" (id 2) (at 97.155 71.12 0)
+      (effects (font (size 1.27 1.27)) hide)
+    )
+    (property "Datasheet" "~" (id 3) (at 97.155 71.12 0)
       (effects (font (size 1.27 1.27)) hide)
     )
@@
   )
   (symbol_instances
+    (path "/0b7c3bb1-e94b-451e-8166-d3776bdc8b16"
+      (reference "#FLG01") (unit 1) (value "PWR_FLAG") (footprint "")
+    )
+    (path "/9ab38907-cc9e-4549-b313-e8f21a7a97ac"
+      (reference "#FLG0101") (unit 1) (value "PWR_FLAG") (footprint "")
+    )
     (path "/1e92318b-3c4f-47e4-bb54-9cbb72ad7d7c"
       (reference "#PWR0101") (unit 1) (value "GND") (footprint "")
@@
     )
     (path "/95e1eb76-8da9-4d97-8379-8facac6c427d"
-      (reference "#PWR?") (unit 1) (value "GND") (footprint "")
+      (reference "#PWR0105") (unit 1) (value "GND") (footprint "")
     )
     (path "/ca007935-a432-42f1-b756-6e4a1ace9956"

Commit message: update
Connections:
- net AGND: no longer U1.8 (AGND)
- net GND: now also U1.8 (AGND)
Other:
- moved on the sheet: NT1
Changed lines of the file:
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@@
   (junction (at 195.58 78.74) (diameter 0) (color 0 0 0 0)
   )
-  (junction (at 165.1 102.87) (diameter 0) (color 0 0 0 0)
-  )
   (junction (at 180.34 71.12) (diameter 0) (color 0 0 0 0)
   )
   (junction (at 147.32 127) (diameter 0) (color 0 0 0 0)
   )
+  (junction (at 165.1 102.235) (diameter 0) (color 0 0 0 0)
+  )
   (junction (at 165.1 88.9) (diameter 0) (color 0 0 0 0)
   )
@@
   (junction (at 91.44 71.12) (diameter 0) (color 0 0 0 0)
   )
+  (junction (at 187.96 78.74) (diameter 0) (color 0 0 0 0)
+  )
+  (junction (at 119.38 104.14) (diameter 0) (color 0 0 0 0)
+  )
+  (junction (at 104.14 71.12) (diameter 0) (color 0 0 0 0)
+  )
+  (junction (at 165.1 96.52) (diameter 0) (color 0 0 0 0)
+  )
   (junction (at 165.1 99.06) (diameter 0) (color 0 0 0 0)
   )
-  (junction (at 187.96 78.74) (diameter 0) (color 0 0 0 0)
-  )
-  (junction (at 119.38 104.14) (diameter 0) (color 0 0 0 0)
-  )
-  (junction (at 104.14 71.12) (diameter 0) (color 0 0 0 0)
-  )
   (wire (pts (xy 116.84 76.2) (xy 116.84 96.52))
     (stroke (width 0) (type default) (color 0 0 0 0))
@@
     (stroke (width 0) (type default) (color 0 0 0 0))
   )
+  (wire (pts (xy 165.1 93.98) (xy 165.1 96.52))
+    (stroke (width 0) (type default) (color 0 0 0 0))
+  )
   (wire (pts (xy 162.56 99.06) (xy 165.1 99.06))
     (stroke (width 0) (type default) (color 0 0 0 0))
@@
     (stroke (width 0) (type default) (color 0 0 0 0))
   )
-  (wire (pts (xy 172.72 99.06) (xy 165.1 99.06))
+  (wire (pts (xy 162.56 93.98) (xy 165.1 93.98))
     (stroke (width 0) (type default) (color 0 0 0 0))
   )
@@
     (stroke (width 0) (type default) (color 0 0 0 0))
   )
+  (wire (pts (xy 165.1 96.52) (xy 165.1 99.06))
+    (stroke (width 0) (type default) (color 0 0 0 0))
+  )
   (wire (pts (xy 88.9 71.12) (xy 91.44 71.12))
     (stroke (width 0) (type default) (color 0 0 0 0))
@@
     (stroke (width 0) (type default) (color 0 0 0 0))
   )
-  (wire (pts (xy 162.56 93.98) (xy 172.72 93.98))
-    (stroke (width 0) (type default) (color 0 0 0 0))
-  )
-  (wire (pts (xy 165.1 99.06) (xy 165.1 102.87))
+  (wire (pts (xy 165.1 99.06) (xy 165.1 102.235))
     (stroke (width 0) (type default) (color 0 0 0 0))
   )
@@
     (stroke (width 0) (type default) (color 0 0 0 0))
   )
-  (wire (pts (xy 172.72 93.98) (xy 172.72 99.06))
-    (stroke (width 0) (type default) (color 0 0 0 0))
-  )
   (wire (pts (xy 165.1 88.9) (xy 167.64 88.9))
     (stroke (width 0) (type default) (color 0 0 0 0))
@@
     (stroke (width 0) (type default) (color 0 0 0 0))
   )
-  (wire (pts (xy 165.1 102.87) (xy 165.1 104.14))
+  (wire (pts (xy 162.56 96.52) (xy 165.1 96.52))
+    (stroke (width 0) (type default) (color 0 0 0 0))
+  )
+  (wire (pts (xy 165.1 102.235) (xy 165.1 104.14))
     (stroke (width 0) (type default) (color 0 0 0 0))
   )
@@
     (stroke (width 0) (type default) (color 0 0 0 0))
   )
-  (wire (pts (xy 178.435 95.885) (xy 182.245 95.885))
+  (wire (pts (xy 196.215 102.87) (xy 200.025 102.87))
     (stroke (width 0) (type default) (color 0 0 0 0))
   )
@@
     )
   )
-  (global_label "AGND" (shape input) (at 162.56 96.52 0) (fields_autoplaced)
+  (global_label "AGND" (shape input) (at 205.105 102.87 0) (fields_autoplaced)
     (effects (font (size 1.27 1.27)) (justify left))
-    (property "Referenzen zwischen Schaltplänen" "${INTERSHEET_REFS}" (id 0) (at 169.8432 96.4406 0)
-      (effects (font (size 1.27 1.27)) (justify left) hide)
-    )
-  )
-  (global_label "AGND" (shape input) (at 187.325 95.885 0) (fields_autoplaced)
-    (effects (font (size 1.27 1.27)) (justify left))
-    (property "Referenzen zwischen Schaltplänen" "${INTERSHEET_REFS}" (id 0) (at 194.6082 95.8056 0)
+    (property "Referenzen zwischen Schaltplänen" "${INTERSHEET_REFS}" (id 0) (at 212.3882 102.7906 0)
       (effects (font (size 1.27 1.27)) (justify left) hide)
     )
@@
     )
   )
-  (symbol (lib_id "power:PWR_FLAG") (at 165.1 102.87 270) (unit 1)
-    (in_bom yes) (on_board yes) (fields_autoplaced)
-    (property "Reference" "#FLG01" (id 0) (at 167.005 102.87 0)
-      (effects (font (size 1.27 1.27)) hide)
-    )
-    (property "Value" "PWR_FLAG" (id 1) (at 168.91 102.8699 90)
-      (effects (font (size 1.27 1.27)) (justify left))
-    )
-    (property "Footprint" "" (id 2) (at 165.1 102.87 0)
-      (effects (font (size 1.27 1.27)) hide)
-    )
-    (property "Datasheet" "~" (id 3) (at 165.1 102.87 0)
+  (symbol (lib_id "power:PWR_FLAG") (at 165.1 102.235 270) (unit 1)
+    (in_bom yes) (on_board yes) (fields_autoplaced)
+    (property "Reference" "#FLG01" (id 0) (at 167.005 102.235 0)
+      (effects (font (size 1.27 1.27)) hide)
+    )
+    (property "Value" "PWR_FLAG" (id 1) (at 168.91 102.2349 90)
+      (effects (font (size 1.27 1.27)) (justify left))
+    )
+    (property "Footprint" "" (id 2) (at 165.1 102.235 0)
+      (effects (font (size 1.27 1.27)) hide)
+    )
+    (property "Datasheet" "~" (id 3) (at 165.1 102.235 0)
       (effects (font (size 1.27 1.27)) hide)
     )
@@
     (pin "2")
   )
-  (symbol (lib_id "power:GND") (at 178.435 95.885 0) (unit 1)
-    (in_bom yes) (on_board yes) (fields_autoplaced)
-    (property "Reference" "#PWR0105" (id 0) (at 178.435 102.235 0)
-      (effects (font (size 1.27 1.27)) hide)
-    )
-    (property "Value" "GND" (id 1) (at 178.435 100.965 0))
-    (property "Footprint" "" (id 2) (at 178.435 95.885 0)
-      (effects (font (size 1.27 1.27)) hide)
-    )
-    (property "Datasheet" "" (id 3) (at 178.435 95.885 0)
+  (symbol (lib_id "power:GND") (at 196.215 102.87 0) (unit 1)
+    (in_bom yes) (on_board yes) (fields_autoplaced)
+    (property "Reference" "#PWR0105" (id 0) (at 196.215 109.22 0)
+      (effects (font (size 1.27 1.27)) hide)
+    )
+    (property "Value" "GND" (id 1) (at 196.215 107.95 0))
+    (property "Footprint" "" (id 2) (at 196.215 102.87 0)
+      (effects (font (size 1.27 1.27)) hide)
+    )
+    (property "Datasheet" "" (id 3) (at 196.215 102.87 0)
       (effects (font (size 1.27 1.27)) hide)
     )
@@
     (pin "1")
   )
-  (symbol (lib_id "Device:NetTie_2") (at 184.785 95.885 0) (unit 1)
+  (symbol (lib_id "Device:NetTie_2") (at 202.565 102.87 0) (unit 1)
     (in_bom no) (on_board yes) (fields_autoplaced)
-    (property "Reference" "NT1" (id 0) (at 184.785 90.805 0))
-    (property "Value" "NetTie_2" (id 1) (at 184.785 93.345 0))
-    (property "Footprint" "NetTie:NetTie-2_SMD_Pad0.5mm" (id 2) (at 184.785 95.885 0)
-      (effects (font (size 1.27 1.27)) hide)
-    )
-    (property "Datasheet" "~" (id 3) (at 184.785 95.885 0)
-      (effects (font (size 1.27 1.27)) hide)
-    )
+    (property "Reference" "NT1" (id 0) (at 202.565 97.79 0))
+    (property "Value" "NetTie_2" (id 1) (at 202.565 100.33 0))
+    (property "Footprint" "NetTie:NetTie-2_SMD_Pad0.5mm" (id 2) (at 202.565 102.87 0)
+      (effects (font (size 1.27 1.27)) hide)
+    )
+    (property "Datasheet" "~" (id 3) (at 202.565 102.87 0)
+      (effects (font (size 1.27 1.27)) hide)
+    )

Commit message: update
Parts:
- added J1, J2: Conn_02x02_Counter_Clockwise, Connector_PinHeader_2.54mm:PinHeader_2x02_P2.54mm_Vertical, symbol Connector_Generic:Conn_02x02_Counter_Clockwise
- added TP1: Vin, TestPoint:TestPoint_Pad_D3.0mm, symbol Connector:TestPoint
- added TP2: Vout, TestPoint:TestPoint_Pad_D3.0mm, symbol Connector:TestPoint
- added TP3, TP4: GND, TestPoint:TestPoint_Pad_D3.0mm, symbol Connector:TestPoint
- added TP5, TP6, TP7, TP8: RCWCTE, Snapeda:RCWCTE_TP420X150, symbol Snapeda:RCWCTE
Connections:
- net EN: now also J1.3 (Pin_3), J1.4 (Pin_4), TP1.1, TP7.1
- net GND: now also J1.1 (Pin_1), J1.2 (Pin_2), J2.1 (Pin_1), J2.2 (Pin_2), TP3.1, TP4.1, TP6.1, TP8.1
- net Vout: now also J2.3 (Pin_3), J2.4 (Pin_4), TP2.1, TP5.1

Commit message: update
Parts:
- C1: value C_Small -> 2.2uF
- C3: value C_Small -> 22uF
- C4, C5: value C_Small -> DNP; now left out of the parts list
- L1: value WE-MAPI_4020 -> 74438356022
Connections:
- net EN renamed Vin
Other:
- note added: "Rosel 4.75k - 3.3V 205k - 5V"
- moved on the sheet: C2
